Commit message: Updates

File: src/xsens_mti_ros2_driver/urdf/MTi_6xx.urdf (robot description, URDF)
Before this commit: robot mti_6xx, 1 links, 0 joints
Links:
- added link vlp16_front; visual mesh filename=package://xsens_mti_ros2_driver/urdf/velodyne-vlp16.stl scale=0.001 0.001 0.001
Joints:
- added joint lidar_imu: type fixed, parent imu_link, child vlp16_front, origin xyz=0.005593697569844 0.002109367719277 -0.072895368036261  rpy=0.0002889054550105368 0.007577368810653143 -0.07620471550025973
